Commit message: 20240914

File: urdf/07-physics.urdf (robot description, URDF)
Before this commit: robot physics, 16 links, 15 joints
Links:
- added link odom
Joints:
- added joint odom_to_base_link: type fixed, parent odom, child base_link

File: urdf/08-macroed.urdf.xacro (robot description, xacro)
@@ -22,4 +22,10 @@
     </inertial>
   </xacro:macro>
+  <link name="odom">
+  </link>
+  <joint name="odom_to_base_link" type="fixed">
+    <parent link="odom"/>
+    <child link="base_link"/>
+  </joint>
   <link name="base_link">
     <visual>
